Commit message: Tried using an external xacro file to fix problem

File: robutlerT3G1_description/urdf/robutlerT3G1.gazebo.xacro (robot description, xacro)
@@ -156,38 +156,6 @@
         <cameraName>camera</cameraName>
         <frameName>camera_rgb_optical_frame</frameName>
-        <imageTopicName>rgb/image_raw</imageTopicName>
-        <cameraInfoTopicName>rgb/camera_info</cameraInfoTopicName>
-        <hackBaseline>0.07</hackBaseline>
-        <distortionK1>0.0</distortionK1>
-        <distortionK2>0.0</distortionK2>
-        <distortionK3>0.0</distortionK3>
-        <distortionT1>0.0</distortionT1>
-        <distortionT2>0.0</distortionT2>
-      </plugin>
-    </sensor>
-  </gazebo>
-  <gazebo reference="camera2_rgb_frame">
-    <sensor type="camera" name="Pi Camera 2">
-      <always_on>true</always_on>
-      <visualize>$(arg camera_visual)</visualize>
-      <camera>
-          <horizontal_fov>1.085595</horizontal_fov>
-          <image>
-              <width>640</width>
-              <height>480</height>
-              <format>R8G8B8</format>
-          </image>
-          <clip>
-              <near>0.03</near>
-              <far>100</far>
-          </clip>
-      </camera>
-      <plugin name="camera2_controller" filename="libgazebo_ros_camera.so">
-        <alwaysOn>true</alwaysOn>
-        <updateRate>30.0</updateRate>
-        <cameraName>camera2</cameraName>
-        <frameName>camera2_rgb_optical_frame</frameName>
-        <imageTopicName>rgb/image_raw2</imageTopicName>
-        <cameraInfoTopicName>rgb/camera_info2</cameraInfoTopicName>
+        <imageTopicName>rgb_fixed/image_raw</imageTopicName>
+        <cameraInfoTopicName>rgb_fixed/camera_info</cameraInfoTopicName>
         <hackBaseline>0.07</hackBaseline>
         <distortionK1>0.0</distortionK1>

File: robutlerT3G1_description/urdf/robutlerT3G1.urdf.xacro (robot description, xacro)
@@ -3,4 +3,5 @@
   <xacro:include filename="$(find robutlerT3G1_description)/urdf/common_properties.xacro"/>
   <xacro:include filename="$(find robutlerT3G1_description)/urdf/robutlerT3G1.gazebo.xacro"/>
+  <xacro:include filename="$(find robutlerT3G1_description)/urdf/rgb_camera.urdf.xacro"/>
   <link name="base_footprint"/>
   <joint name="base_joint" type="fixed">
@@ -209,4 +210,5 @@
   <child link="rotating_camera_base_link"/>
   <axis xyz="0 0 1" />
+  <limit effort="1000.0" lower="0.35" upper="0.6" velocity="0.5" />
 </joint>
 <!-- Rotating Camera base -->
@@ -221,5 +223,5 @@
 </link>
 <!-- Joint for Rotating Camera -->
-<joint name="rotating_camera_joint" type="continuous">
+<joint name="rotating_camera_joint" type="fixed">
   <origin xyz="0 0 0.05" rpy="0 0 0"/>
   <parent link="rotating_camera_base_link"/>
@@ -229,28 +231,11 @@
 </joint>
 <!-- new camera -->
-  <joint name="camera2_joint" type="fixed">
-    <origin xyz="0.02 0 0" rpy="0 0 0"/>
-    <parent link="rotating_camera_link"/>
-    <child link="camera2_link"/>
-  </joint>
-  <link name="camera2_link">
-    <collision>
-      <origin xyz="0.005 0.011 0.013" rpy="0 0 0"/>
-      <geometry>
-        <box size="0.015 0.030 0.027"/>
-      </geometry>
-    </collision>
-  </link>
-  <joint name="camera2_rgb_joint" type="fixed">
-    <origin xyz="0.003 0.011 0.009" rpy="0 0 0"/>
-    <parent link="camera2_link"/>
-    <child link="camera2_rgb_frame"/>
-  </joint>
-  <link name="camera2_rgb_frame"/>
-  <joint name="camera2_rgb_optical_joint" type="fixed">
-    <origin xyz="0 0 0" rpy="-1.57 0 -1.57"/>
-    <parent link="camera2_rgb_frame"/>
-    <child link="camera2_rgb_optical_frame"/>
-  </joint>
-  <link name="camera2_rgb_optical_frame"/>
+    <xacro:rgb_camera parent="rotating_camera_link" prefix="rgb_rotating" color_gazebo="White">
+        <origin xyz="0.015 0 0.012" rpy="0 0 0" />
+        <color_rgb_rviz>
+            <material name="white">
+                <color rgba="1.0 1.0 1.0 1" />
+            </material>
+        </color_rgb_rviz>
+    </xacro:rgb_camera>
 </robot>
