Commit message: #1 adding a second camera

File: robutlerT3G1_description/urdf/common_properties.xacro (robot description, xacro)
@@ -32,3 +32,6 @@
     <color rgba="1.0 1.0 1.0 1.0"/>
   </material>
+  <material name="invisible">
+    <color rgba="1.0 1.0 1.0 0.05"/>
+  </material>
 </robot>

File: robutlerT3G1_description/urdf/robutlerT3G1.gazebo.xacro (robot description, xacro)
@@ -6,4 +6,10 @@
   <gazebo reference="base_link">
     <material>Gazebo/SkyBlue </material>
+  </gazebo>
+  <gazebo reference="rotating_camera_base_link">
+    <material>Gazebo/SkyBlue </material>
+  </gazebo>
+  <gazebo reference="rotating_camera_link">
+    <material>Gazebo/White </material>
   </gazebo>
   <gazebo reference="wheel_left_link">

File: robutlerT3G1_description/urdf/robutlerT3G1.urdf.xacro (robot description, xacro)
@@ -194,48 +194,59 @@
   </joint>
   <link name="camera_rgb_optical_frame"/>
-<!-- Rotating Camera base -->
-<link name="rotating_camera_base_link">
-  <visual>
-    <geometry>
-      <cylinder length="0.05" radius="0.01" />
-    </geometry>
-    <origin xyz="0 0 0.025" rpy="0 0 0" />
-    <material name="blue" />
-  </visual>
-</link>
-<!-- Joint for Rotating Camera base -->
-<joint name="rotating_camera_base_joint" type="fixed">
-  <origin xyz="-0.15 0 0.09" rpy="0 0 0"/>
-  <parent link="base_link"/>
-  <child link="rotating_camera_base_link"/>
-  <axis xyz="0 0 1" />
-  <limit effort="1000.0" lower="0.35" upper="0.6" velocity="0.5" />
-</joint>
-<!-- Rotating Camera base -->
-<link name="rotating_camera_link">
-  <visual>
-    <geometry>
-      <sphere radius="0.02" />
-    </geometry>
-    <origin xyz="0 0 0" rpy="0 0 0" />
-    <material name="white" />
-  </visual>
-</link>
-<!-- Joint for Rotating Camera -->
-<joint name="rotating_camera_joint" type="fixed">
-  <origin xyz="0 0 0.05" rpy="0 0 0"/>
-  <parent link="rotating_camera_base_link"/>
-  <child link="rotating_camera_link"/>
-  <axis xyz="0 1 0"/>
-  <limit effort="1000.0" lower="0.35" upper="0.6" velocity="0.5" />
-</joint>
-<!-- new camera -->
-    <xacro:rgb_camera parent="rotating_camera_link" prefix="rgb_rotating" color_gazebo="White">
-        <origin xyz="0.015 0 0.012" rpy="0 0 0" />
-        <color_rgb_rviz>
-            <material name="white">
-                <color rgba="1.0 1.0 1.0 1" />
-            </material>
-        </color_rgb_rviz>
-    </xacro:rgb_camera>
+  <!-- Rotating Camera base -->
+  <link name="rotating_camera_base_link">
+    <visual>
+      <geometry>
+        <cylinder length="0.05" radius="0.01" />
+      </geometry>
+      <origin xyz="0 0 0.025" rpy="0 0 0" />
+      <material name="blue" />
+    </visual>
+    <inertial>
+      <mass value="0.04" />
+      <origin xyz="0 0 0" />
+      <inertia ixx="0.001" ixy="0.0" ixz="0.0"
+               iyy="0.001" iyz="0.0"
+               izz="0.001" />
+    </inertial>
+  </link>
+  <!-- Joint for Rotating Camera base -->
+  <joint name="rotating_camera_base_joint" type="continuous">
+    <origin xyz="-0.15 0 0.09" rpy="0 0 0"/>
+    <parent link="base_link"/>
+    <child link="rotating_camera_base_link"/>
+    <axis xyz="0 0 1" />
+  </joint>
+  <!-- Rotating Camera support -->
+  <link name="rotating_camera_link">
+    <visual>
+      <geometry>
+        <sphere radius="0.02" />
+      </geometry>
+      <origin xyz="0 0 0" rpy="0 0 0" />
+      <material name="white" />
+    </visual>
+    <inertial>
+      <mass value="0.04" />
+      <origin xyz="0 0 0" />
+      <inertia ixx="0.001" ixy="0.0" ixz="0.0"
+               iyy="0.001" iyz="0.0"
+               izz="0.001" />
+    </inertial>
+  </link>
+  <!-- Joint for Rotating Camera -->
+  <joint name="rotating_camera_joint" type="revolute">
+    <origin xyz="0 0 0.05" rpy="0 -1.57 0"/>
+    <parent link="rotating_camera_base_link"/>
+    <child link="rotating_camera_link"/>
+    <axis xyz="0 1 0"/>
+    <limit effort="1000.0" lower="0" upper="2.36" velocity="0.5" />
+  </joint>
+  <!-- new camera -->
+  <xacro:rgb_camera parent="rotating_camera_link" prefix="rgb_rotating" color_gazebo="White">
+      <origin xyz="0.015 0 0.012" rpy="0 0 0" />
+      <color_rgb_rviz>
+          <material name="white"/>
+      </color_rgb_rviz>
+  </xacro:rgb_camera>
 </robot>
