Commit message: #11 Reduced model complexity and reduced models in the world

File: robutler1_description/urdf/robutler1.gazebo.xacro (robot description, xacro)
@@ -8,7 +8,4 @@
   </gazebo>
   <gazebo reference="rotating_camera_base_link">
-    <material>Gazebo/SkyBlue </material>
-  </gazebo>
-  <gazebo reference="rotating_camera_link">
     <material>Gazebo/White </material>
   </gazebo>
@@ -159,5 +156,5 @@
       <plugin name="camera_controller" filename="libgazebo_ros_camera.so">
         <alwaysOn>true</alwaysOn>
-        <updateRate>30.0</updateRate>
+        <updateRate>20.0</updateRate>
         <cameraName>camera</cameraName>
         <frameName>camera_rgb_optical_frame</frameName>
@@ -173,3 +170,37 @@
     </sensor>
   </gazebo>
+<!--2nd camera-->
+<!--link : https://www.raspberrypi.org/documentation/hardware/camera/-->
+  <gazebo reference="camera2_rgb_frame">
+    <sensor type="camera" name="Pi Camera">
+      <always_on>true</always_on>
+      <visualize>$(arg camera_visual)</visualize>
+      <camera>
+          <horizontal_fov>1.085595</horizontal_fov>
+          <image>
+              <width>640</width>
+              <height>480</height>
+              <format>R8G8B8</format>
+          </image>
+          <clip>
+              <near>0.03</near>
+              <far>100</far>
+          </clip>
+      </camera>
+      <plugin name="camera_controller" filename="libgazebo_ros_camera.so">
+        <alwaysOn>true</alwaysOn>
+        <updateRate>20.0</updateRate>
+        <cameraName>camera2</cameraName>
+        <frameName>camera2_rgb_optical_frame</frameName>
+        <imageTopicName>rgb_rotating/image_raw</imageTopicName>
+        <cameraInfoTopicName>rgb_rotating/camera_info</cameraInfoTopicName>
+        <hackBaseline>0.07</hackBaseline>
+        <distortionK1>0.0</distortionK1>
+        <distortionK2>0.0</distortionK2>
+        <distortionK3>0.0</distortionK3>
+        <distortionT1>0.0</distortionT1>
+        <distortionT2>0.0</distortionT2>
+      </plugin>
+    </sensor>
+  </gazebo>
 </robot>

File: robutler1_description/urdf/robutler1.urdf.xacro (robot description, xacro)
@@ -3,5 +3,4 @@
   <xacro:include filename="$(find robutler1_description)/urdf/common_properties.xacro"/>
   <xacro:include filename="$(find robutler1_description)/urdf/robutler1.gazebo.xacro"/>
-  <xacro:include filename="$(find robutler1_description)/urdf/rgb_camera.urdf.xacro"/>
   <link name="base_footprint"/>
   <joint name="base_joint" type="fixed">
@@ -201,5 +200,5 @@
       </geometry>
       <origin xyz="0 0 0.025" rpy="0 0 0" />
-      <material name="blue" />
+      <material name="white" />
     </visual>
     <inertial>
@@ -218,35 +217,29 @@
     <axis xyz="0 0 1" />
   </joint>
-  <!-- Rotating Camera support -->
-  <link name="rotating_camera_link">
-    <visual>
-      <geometry>
-        <sphere radius="0.02" />
-      </geometry>
-      <origin xyz="0 0 0" rpy="0 0 0" />
-      <material name="white" />
-    </visual>
-    <inertial>
-      <mass value="0.04" />
-      <origin xyz="0 0 0" />
-      <inertia ixx="0.001" ixy="0.0" ixz="0.0"
-               iyy="0.001" iyz="0.0"
-               izz="0.001" />
-    </inertial>
-  </link>
-  <!-- Joint for Rotating Camera -->
-  <joint name="rotating_camera_joint" type="revolute">
-    <origin xyz="0 0 0.05" rpy="0 -1.57 0"/>
+  <!-- new camera -->
+  <joint name="camera2_joint" type="fixed">
+    <origin xyz="0.073 -0.011 0.084" rpy="0 0 0"/>
     <parent link="rotating_camera_base_link"/>
-    <child link="rotating_camera_link"/>
-    <axis xyz="0 1 0"/>
-    <limit effort="1000.0" lower="0" upper="2.36" velocity="0.5" />
-  </joint>
-  <!-- new camera -->
-  <xacro:rgb_camera parent="rotating_camera_link" prefix="rgb_rotating" color_gazebo="White">
-      <origin xyz="0.015 0 0.012" rpy="0 0 0" />
-      <color_rgb_rviz>
-          <material name="white"/>
-      </color_rgb_rviz>
-  </xacro:rgb_camera>
+    <child link="camera2_link"/>
+  </joint>
+  <link name="camera2_link">
+    <collision>
+      <origin xyz="0.005 0.011 0.013" rpy="0 0 0"/>
+      <geometry>
+        <box size="0.015 0.030 0.027"/>
+      </geometry>
+    </collision>
+  </link>
+  <joint name="camera2_rgb_joint" type="fixed">
+    <origin xyz="0.003 0.011 0.009" rpy="0 0 0"/>
+    <parent link="camera2_link"/>
+    <child link="camera2_rgb_frame"/>
+  </joint>
+  <link name="camera2_rgb_frame"/>
+  <joint name="camera2_rgb_optical_joint" type="fixed">
+    <origin xyz="0 0 0" rpy="-1.57 0 -1.57"/>
+    <parent link="camera2_rgb_frame"/>
+    <child link="camera2_rgb_optical_frame"/>
+  </joint>
+  <link name="camera2_rgb_optical_frame"/>
 </robot>
