Commit message: #13 added robotic arm from he turtlebot in the model

File: robutler1_description/urdf/robutlerv2.gazebo.xacro (robot description, xacro)
@@ -5,12 +5,9 @@
   <xacro:arg name="imu_visual"    default="false"/>
   <gazebo reference="base_link">
-    <material>Gazebo/SkyBlue </material>
-  </gazebo>
-  <gazebo reference="rotating_camera_base_link">
-    <material>Gazebo/White </material>
+    <material>Gazebo/DarkGrey</material>
   </gazebo>
   <gazebo reference="wheel_left_link">
-    <mu1>0.1</mu1>
-    <mu2>0.1</mu2>
+    <mu1>10000</mu1>
+    <mu2>10000</mu2>
     <kp>500000.0</kp>
     <kd>10.0</kd>
@@ -21,6 +18,6 @@
   </gazebo>
   <gazebo reference="wheel_right_link">
-    <mu1>0.1</mu1>
-    <mu2>0.1</mu2>
+    <mu1>10000</mu1>
+    <mu2>10000</mu2>
     <kp>500000.0</kp>
     <kd>10.0</kd>
@@ -106,5 +103,5 @@
   </gazebo>
   <gazebo reference="base_scan">
-    <material>Gazebo/Gold</material>
+    <material>Gazebo/FlatBlack</material>
     <sensor type="ray" name="lds_lfcd_sensor">
       <pose>0 0 0 0 0 0</pose>
@@ -156,9 +153,9 @@
       <plugin name="camera_controller" filename="libgazebo_ros_camera.so">
         <alwaysOn>true</alwaysOn>
-        <updateRate>20.0</updateRate>
+        <updateRate>30.0</updateRate>
         <cameraName>camera</cameraName>
         <frameName>camera_rgb_optical_frame</frameName>
-        <imageTopicName>rgb_fixed/image_raw</imageTopicName>
-        <cameraInfoTopicName>rgb_fixed/camera_info</cameraInfoTopicName>
+        <imageTopicName>rgb/image_raw</imageTopicName>
+        <cameraInfoTopicName>rgb/camera_info</cameraInfoTopicName>
         <hackBaseline>0.07</hackBaseline>
         <distortionK1>0.0</distortionK1>
@@ -170,3 +167,37 @@
     </sensor>
   </gazebo>
+  <!--2nd camera-->
+  <!--link : https://www.raspberrypi.org/documentation/hardware/camera/-->
+  <gazebo reference="camera2_rgb_frame">
+    <sensor type="camera" name="Pi Camera">
+      <always_on>true</always_on>
+      <visualize>$(arg camera_visual)</visualize>
+      <camera>
+          <horizontal_fov>1.085595</horizontal_fov>
+          <image>
+              <width>640</width>
+              <height>480</height>
+              <format>R8G8B8</format>
+          </image>
+          <clip>
+              <near>0.03</near>
+              <far>100</far>
+          </clip>
+      </camera>
+      <plugin name="camera_controller" filename="libgazebo_ros_camera.so">
+        <alwaysOn>true</alwaysOn>
+        <updateRate>20.0</updateRate>
+        <cameraName>camera2</cameraName>
+        <frameName>camera2_rgb_optical_frame</frameName>
+        <imageTopicName>rgb_rotating/image_raw</imageTopicName>
+        <cameraInfoTopicName>rgb_rotating/camera_info</cameraInfoTopicName>
+        <hackBaseline>0.07</hackBaseline>
+        <distortionK1>0.0</distortionK1>
+        <distortionK2>0.0</distortionK2>
+        <distortionK3>0.0</distortionK3>
+        <distortionT1>0.0</distortionT1>
+        <distortionT2>0.0</distortionT2>
+      </plugin>
+    </sensor>
+  </gazebo>
 </robot>

File: robutler1_description/urdf/robutlerv2.urdf.xacro (robot description, xacro)
@@ -1,6 +1,6 @@
 <?xml version="1.0" ?>
-<robot name="turtlebot3_waffle_pi" xmlns:xacro="http://ros.org/wiki/xacro">
+<robot name="turtlebot3_waffle_pi_for_open_manipulator" xmlns:xacro="http://ros.org/wiki/xacro">
   <xacro:include filename="$(find robutler1_description)/urdf/common_properties.xacro"/>
-  <xacro:include filename="$(find robutler1_description)/urdf/robutler1.gazebo.xacro"/>
+  <xacro:include filename="$(find robutler1_description)/urdf/robutlerv2.gazebo.xacro"/>
   <link name="base_footprint"/>
   <joint name="base_joint" type="fixed">
@@ -9,12 +9,11 @@
     <origin xyz="0 0 0.010" rpy="0 0 0"/>
   </joint>
-  <!-- base link -->
   <link name="base_link">
     <visual>
       <origin xyz="-0.064 0 0.0" rpy="0 0 0"/>
       <geometry>
-        <mesh filename="package://turtlebot3_description/meshes/bases/waffle_pi_base.stl" scale="0.001 0.001 0.001"/>
+        <mesh filename="package://turtlebot3_description/meshes/bases/waffle_pi_base_for_open_manipulator.stl" scale="0.001 0.001 0.001"/>
       </geometry>
-      <material name="blue"/>
+      <material name="light_black"/>
     </visual>
     <collision>
@@ -25,12 +24,14 @@
     </collision>
     <inertial>
-      <origin xyz="0 0 0" rpy="0 0 0"/>
-      <mass value="1.3729096e+00"/>
-      <inertia ixx="8.7002718e-03" ixy="-4.7576583e-05" ixz="1.1160499e-04"
+      <origin xyz="0.0 0 0.0" rpy="0 0 0"/>
+      <mass value="1.6329594e+00"/>
+      <inertia ixx="1.0" ixy="0.0" ixz="0.0"
+               iyy="1.0" iyz="0.0"
+               izz="1.0" />
+      <!-- <inertia ixx="8.7002718e-03" ixy="-4.7576583e-05" ixz="1.1160499e-04"
                iyy="8.6195418e-03" iyz="-3.5422299e-06"
-               izz="1.4612727e-02" />
+               izz="1.4612727e-02" />                -->
     </inertial>
   </link>
-  <!-- left wheel and left wheel joint -->
   <joint name="wheel_left_joint" type="continuous">
     <parent link="base_link"/>
@@ -61,5 +62,4 @@
       </inertial>
   </link>
-  <!-- right wheel and right wheel joint -->
   <joint name="wheel_right_joint" type="continuous">
     <parent link="base_link"/>
@@ -77,5 +77,5 @@
     </visual>
     <collision>
-      <origin xyz="0 0 0" rpy="0 0 0"/>
+      <origin xyz="0 0.001 0" rpy="0 0 0"/>
       <geometry>
         <cylinder length="0.018" radius="0.033"/>
@@ -90,5 +90,4 @@
       </inertial>
   </link>
-  <!-- Right back wheel and joint -->
   <joint name="caster_back_right_joint" type="fixed">
     <parent link="base_link"/>
@@ -111,5 +110,4 @@
     </inertial>
   </link>
-  <!-- Left back wheel and joint -->
   <joint name="caster_back_left_joint" type="fixed">
     <parent link="base_link"/>
@@ -132,5 +130,4 @@
     </inertial>
   </link>
-  <!-- IMU and joint -->
   <joint name="imu_joint" type="fixed">
     <parent link="base_link"/>
@@ -139,9 +136,8 @@
   </joint>
   <link name="imu_link"/>
-  <!-- Lidar and joint -->
   <joint name="scan_joint" type="fixed">
     <parent link="base_link"/>
     <child link="base_scan"/>
-    <origin xyz="-0.064 0 0.122" rpy="0 0 0"/>
+    <origin xyz="-0.024 0 0.122" rpy="0 0 0"/>
   </joint>
   <link name="base_scan">
@@ -156,5 +152,5 @@
       <origin xyz="0.015 0 -0.0065" rpy="0 0 0"/>
       <geometry>
-        <cylinder length="0.0315" radius="0.055"/>
+        <cylinder length="0.0315" radius="0.045"/>
       </geometry>
     </collision>
@@ -167,5 +163,4 @@
     </inertial>
   </link>
-  <!-- old camera -->
   <joint name="camera_joint" type="fixed">
     <origin xyz="0.073 -0.011 0.084" rpy="0 0 0"/>
