Commit message: #15 Addede the robot arm to the robot. Not moving yet, tho

File: robutler1_description/urdf/open_manipulator_x.urdf.xacro (robot description, xacro)
@@ -12,5 +12,5 @@
         <mesh filename="package://robutler1_description/meshes/chain_link1.stl" scale="0.001 0.001 0.001"/>
       </geometry>
-      <material name="grey"/>
+      <material name="white"/>
     </visual>
     <collision>
@@ -43,5 +43,5 @@
         <mesh filename="package://robutler1_description/meshes/chain_link2.stl" scale="0.001 0.001 0.001"/>
       </geometry>
-      <material name="grey"/>
+      <material name="white"/>
     </visual>
     <collision>
@@ -74,5 +74,5 @@
         <mesh filename="package://robutler1_description/meshes/chain_link3.stl" scale="0.001 0.001 0.001"/>
       </geometry>
-      <material name="grey"/>
+      <material name="white"/>
     </visual>
     <collision>
@@ -105,5 +105,5 @@
         <mesh filename="package://robutler1_description/meshes/chain_link4.stl" scale="0.001 0.001 0.001"/>
       </geometry>
-      <material name="grey"/>
+      <material name="white"/>
     </visual>
     <collision>
@@ -136,5 +136,5 @@
         <mesh filename="package://robutler1_description/meshes/chain_link5.stl" scale="0.001 0.001 0.001"/>
       </geometry>
-      <material name="grey"/>
+      <material name="white"/>
     </visual>
     <collision>
@@ -163,5 +163,5 @@
         <mesh filename="package://robutler1_description/meshes/chain_link_grip_l.stl" scale="0.001 0.001 0.001"/>
       </geometry>
-      <material name="grey"/>
+      <material name="white"/>
     </visual>
     <collision>
@@ -194,5 +194,5 @@
         <mesh filename="package://robutler1_description/meshes/chain_link_grip_r.stl" scale="0.001 0.001 0.001"/>
       </geometry>
-      <material name="grey"/>
+      <material name="white"/>
     </visual>
     <collision>

File: robutler1_description/urdf/robutlerv2.gazebo.xacro (robot description, xacro)
@@ -5,5 +5,5 @@
   <xacro:arg name="imu_visual"    default="false"/>
   <gazebo reference="base_link">
-    <material>Gazebo/DarkGrey</material>
+    <material>Gazebo/SkyBlue</material>
   </gazebo>
   <gazebo reference="wheel_left_link">
@@ -103,5 +103,5 @@
   </gazebo>
   <gazebo reference="base_scan">
-    <material>Gazebo/FlatBlack</material>
+    <material>Gazebo/Gold</material>
     <sensor type="ray" name="lds_lfcd_sensor">
       <pose>0 0 0 0 0 0</pose>
@@ -156,5 +156,5 @@
         <cameraName>camera</cameraName>
         <frameName>camera_rgb_optical_frame</frameName>
-        <imageTopicName>rgb/image_raw</imageTopicName>
+        <imageTopicName>rgb_fixed/image_raw</imageTopicName>
         <cameraInfoTopicName>rgb/camera_info</cameraInfoTopicName>
         <hackBaseline>0.07</hackBaseline>

File: robutler1_description/urdf/robutlerv2.urdf.xacro (robot description, xacro)
@@ -15,5 +15,5 @@
         <mesh filename="package://turtlebot3_description/meshes/bases/waffle_pi_base_for_open_manipulator.stl" scale="0.001 0.001 0.001"/>
       </geometry>
-      <material name="light_black"/>
+      <material name="blue"/>
     </visual>
     <collision>
@@ -147,5 +147,5 @@
         <mesh filename="package://turtlebot3_description/meshes/sensors/lds.stl" scale="0.001 0.001 0.001"/>
       </geometry>
-      <material name="dark"/>
+      <material name="white"/>
     </visual>
     <collision>

File: robutler1_description/urdf/turtlebot3_manipulation_robot.urdf.xacro (robot description, xacro)
@@ -2,5 +2,5 @@
 <robot name="turtlebot3_manipulation" xmlns:xacro="http://ros.org/wiki/xacro">
   <!-- Include TurtleBot3 Waffle URDF -->
-  <xacro:include filename="$(find robutler1_description)/urdf/robutler1.urdf.xacro"/>
+  <xacro:include filename="$(find robutler1_description)/urdf/robutlerv2.urdf.xacro"/>
   <!-- Include OpenMANIPULATOR URDF -->
   <xacro:include filename="$(find robutler1_description)/urdf/open_manipulator_x.urdf.xacro"/>
